File: kicad-project/project/_autosave-ShieldArduino_Semaforo.kicad_sch (KiCad schematic)
At the start: 65 parts, among them IC2 TPS563200DDCR, J1 Conn_01x15, K1 RELAY, P1 Power, P2 Analog, P3 Digital, P4 Digital, P5 CONN_01X01, P6 CONN_01X01, P7 CONN_01X01, P8 CONN_01X01, Q1 PMOS, Q2 NMOS, Q3 NMOS, Q4 NMOS, Q5 NMOS, U1 MCP2542FD-E/MF, U2 LM321

Commit message: kicad-pcb-layout-v0.9
Other:
- moved on the sheet: D1, D11, D12, D13, D2, D3, D4
