File: kicad-project/project/ShieldArduino_Semaforo.kicad_pcb (KiCad board)
At the start: 4 copper layers, 68.6 x 53.3 mm, 65 parts, among them IC2 TPS563200DDCR, J1 Conn_01x15, K1 RELAY, P1 Power, P2 Analog, P3 Digital, P4 Digital, P5 CONN_01X01, P6 CONN_01X01, P7 CONN_01X01, P8 CONN_01X01, Q1 PMOS, Q2 NMOS, Q3 NMOS, Q4 NMOS, Q5 NMOS, U1 MCP2542FD-E/MF, U2 LM321

Commit message: kicad-pcb-layout-v0.9
Connections:
- J1 pad 11: /12V_in -> /throttle_in
- J1 pad 5: /throttle_in -> /12V_in
Routing:
- net /brake_in: track 0.00 -> 57.3 mm, vias 0 -> 2
- net /throttle_in: track 0.00 -> 48.6 mm, vias 0 -> 2
- net /reverse: track 66.3 -> 104.9 mm, vias 4 -> 5
- net +5V: track 51.3 -> 88.0 mm, vias 0 -> 2
- net /relay_out: track 41.6 -> 74.7 mm
- net /inverter_signal_5V: track 41.2 -> 73.3 mm
- net /12V_in: track 1.48 -> 27.9 mm, vias 1 -> 0
- net /low_speed: track 73.1 -> 95.2 mm, vias 4 -> 5
- net /high_speed: track 75.6 -> 92.9 mm, vias 6 -> 7
- net / relay_in: track 61.7 -> 64.8 mm, vias 1 -> 2
- net /12V_in_protected: track 67.7 -> 68.8 mm
Other:
- board text removed: "F2"

Commit message: kicad-pcb-layout-v0.9.1
Parts:
- moved D5 1.36 mm to (115.8, 89.6)
- moved C2 0.11 mm to (144.2, 114.8)
Routing:
- net / relay_in: track 64.8 -> 81.5 mm
- net /throttle_in: track 48.6 -> 54.6 mm
- net /relay_out: track 74.7 -> 79.0 mm
- net /5V_unfused: track 25.7 -> 24.2 mm
- net GND: track 3.67 -> 4.78 mm, vias 4 -> 5
- net /EX_CAN+: track 21.3 -> 22.3 mm

Commit message: kicad-pcb-layout-v1.0
Parts:
- removed J1: Conn_01x15, footprint:L17HTHES4R1C
- added J2: Conn_01x18, footprint:M80-54016YY, F.Cu at (116.9, 118.4)
- moved D1 38.6 mm to (124.1, 113.8)
- moved D2 34.8 mm to (124.1, 111.5)
- moved D3 31.2 mm to (124.1, 109.1)
- moved D4 28.0 mm to (124.1, 106.8)
- moved D11 25.3 mm to (124.1, 104.4)
- moved C7 24.2 mm to (127.9, 88.9)
- moved R3 24.2 mm to (126.8, 94.0)
- moved R4 24.2 mm to (124.6, 84.7)
- moved R5 24.2 mm to (124.6, 88.0)
- moved C2 24.2 mm to (127.6, 97.3)
- moved R1 24.2 mm to (124.3, 93.1)
- moved R2 24.2 mm to (124.3, 96.5)
- moved R6 24.2 mm to (127.1, 85.6)
- moved D12 20.8 mm to (130.7, 108.2)
- moved D13 20.7 mm to (130.7, 110.5)
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Routing:
- net /brake_in_3V3: track 35.7 -> 80.6 mm
- net /high_speed: track 92.9 -> 53.6 mm, vias 7 -> 3
- net /throttle_in_3V3: track 26.3 -> 62.5 mm
- net /12V_in: track 27.9 -> 57.0 mm, vias 0 -> 1
- net /brake_in: track 57.3 -> 33.2 mm, vias 2 -> 0
- net /low_speed: track 95.2 -> 72.8 mm, vias 5 -> 3
- net /inverter_signal_5V: track 73.3 -> 52.6 mm
- net / relay_in: track 81.5 -> 63.5 mm, vias 2 -> 1
- net /reverse: track 104.9 -> 88.8 mm, vias 5 -> 3
- net /12V_in_protected: track 68.8 -> 56.0 mm
- net /throttle_in: track 54.6 -> 42.8 mm, vias 2 -> 3
- net /Vin: track 35.6 -> 24.4 mm, vias 0 -> 1
- net /relay_out: track 79.0 -> 86.4 mm
- net /EX_CAN-: track 23.4 -> 21.6 mm
- net /A5(SCL): track 1.81 -> 0.00 mm
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
Commit message: kicad-pcb-layout-v1.0.1
Parts:
- added C3: 100n, Capacitor_SMD:C_0805_2012Metric_Pad1.18x1.45mm_HandSolder, F.Cu at (206.2, 64.8)
- added C5: 220p, Capacitor_SMD:C_0805_2012Metric_Pad1.18x1.45mm_HandSolder, F.Cu at (206.2, 67.8)
- added D6: D_Small, footprint:SODFL3618X100N, F.Cu at (200.2, 81.7)
- added IC1: TLIN1039DDFRQ1, footprint:SOT65P280X110-8N, F.Cu at (191.8, 81.8)
- added R12: 10k, Resistor_SMD:R_0805_2012Metric_Pad1.20x1.40mm_HandSolder, F.Cu at (206.2, 70.8)
- added R13: 1k, Resistor_SMD:R_0805_2012Metric_Pad1.20x1.40mm_HandSolder, F.Cu at (206.2, 73.7)
Connections:
- J2 pad 15: GND -> /TLIN
- J2 pad 17: GND -> /A4(SDA)
- J2 pad 18: GND -> /A5(SCL)

Commit message: kicad-pcb-layout-v1.0.3
Parts:
- added C6: 100n, Capacitor_SMD:C_0805_2012Metric_Pad1.18x1.45mm_HandSolder, F.Cu at (154.4, 64.9)
- added IC3: MCP4901T-E_MS, footprint:SOP65P490X110-8N, F.Cu at (155.6, 56.7)
- added R21: 200, Resistor_SMD:R_0603_1608Metric_Pad0.98x0.95mm_HandSolder, F.Cu at (159.0, 60.2)
- added R22: 5k, Resistor_SMD:R_0603_1608Metric_Pad0.98x0.95mm_HandSolder, F.Cu at (159.0, 62.7)
- added R23: 5k, Resistor_SMD:R_0603_1608Metric_Pad0.98x0.95mm_HandSolder, F.Cu at (159.0, 65.2)
- added U3: LM4040DBZ-2.0, Package_TO_SOT_SMD:SOT-23, F.Cu at (154.4, 61.2)
- moved C3 23.9 mm to (201.1, 88.1), turned to -90 degrees
- moved R12 22.6 mm to (185.6, 80.0), turned to -90 degrees
- moved C5 20.5 mm to (206.3, 88.3), turned to -90 degrees
- moved D6 7.95 mm to (202.8, 74.2), turned to 90 degrees
- moved R13 6.23 mm to (202.8, 79.0), turned to -90 degrees
- moved C2 4.16 mm to (124.1, 95.1)
- moved R1 4.16 mm to (120.8, 90.9)
- moved R2 4.16 mm to (120.8, 94.2)
- moved R3 4.16 mm to (123.3, 91.8)
- moved R6 4.02 mm to (123.3, 84.3)
- moved C7 4.02 mm to (124.1, 87.6)
- moved R4 4.02 mm to (120.8, 83.4)
- moved R5 4.02 mm to (120.8, 86.7)
Connections:
- P4 pad 1: /7 -> /STM_LDAC
- P4 pad 2: /6(**) -> /STM_DAC_IN
Routing:
- net /throttle_in: track 42.8 -> 47.2 mm
- net /brake_in_3V3: track 80.6 -> 83.9 mm
- net /reverse: track 88.8 -> 87.5 mm
- net /throttle_in_3V3: track 62.5 -> 63.6 mm
- net /low_speed: track 72.8 -> 72.1 mm

Commit message: kicad-pcb-layout-v1.0.4
Parts:
- added JP1: Jumper_2_Small_Bridged, Jumper:SolderJumper-2_P1.3mm_Bridged_RoundedPad1.0x1.5mm, F.Cu at (96.6, 87.0)
- added JP2: Jumper_2_Small_Open, Jumper:SolderJumper-2_P1.3mm_Open_RoundedPad1.0x1.5mm, F.Cu at (94.0, 86.9)
- moved R22 68.2 mm to (94.4, 84.5), turned to 180 degrees
- moved U3 65.2 mm to (96.3, 90.7), turned to -90 degrees
- moved R23 65.1 mm to (98.8, 89.9), turned to 90 degrees
- moved IC3 63.1 mm to (97.8, 82.0), turned to -90 degrees
- moved R21 61.8 mm to (99.9, 78.1)
- moved C6 56.0 mm to (100.6, 80.8), turned to -90 degrees
- moved C5 38.5 mm to (167.8, 88.1), turned to 180 degrees
- moved D6 33.1 mm to (170.8, 82.7), turned to -90 degrees
- moved R13 30.6 mm to (173.0, 85.5)
- moved C3 30.4 mm to (170.7, 86.9)
- moved IC1 24.5 mm to (167.5, 85.4)
- moved R12 22.1 mm to (164.2, 85.4), turned to 90 degrees
Routing:
- net /TLIN: track 0.00 -> 90.7 mm, vias 0 -> 1
- net +3V3: track 0.00 -> 57.0 mm, vias 0 -> 1
- net /12V_in_protected: track 56.0 -> 94.8 mm
- net /reverse: track 87.5 -> 64.5 mm
- net /UART_RX: track 0.00 -> 13.5 mm
- net /UART_TX: track 0.00 -> 13.3 mm, vias 0 -> 1
- net Net-(IC3-VREF): track 0.00 -> 5.02 mm
- net Net-(D6-K): track 0.00 -> 4.34 mm
- net Net-(JP1-B): track 0.00 -> 4.21 mm
- net Net-(IC1-EN): track 0.00 -> 2.39 mm
- net /inverter_signal_3V3: track 94.7 -> 92.4 mm
- net /STM_DAC_IN: track 0.45 -> 2.54 mm
- net +5V: track 89.7 -> 91.6 mm
- net /STM_LDAC: track 0.00 -> 1.68 mm

Commit message: kicad-pcb-layout-v1.0.5
Parts:
- moved C6 108.1 mm to (207.1, 100.0)
- moved R23 108.1 mm to (205.2, 109.1)
- moved U3 108.1 mm to (202.7, 109.9)
- moved IC3 108.1 mm to (204.3, 101.3)
- moved JP1 108.1 mm to (203.0, 106.2)
- moved JP2 108.1 mm to (200.4, 106.2)
- moved R21 108.1 mm to (206.3, 97.3)
- moved R22 108.1 mm to (200.8, 103.7)
Routing:
- net /UART_RX: track 13.5 -> 21.9 mm
- net +5V: track 91.6 -> 98.4 mm
- net / relay_in: track 63.5 -> 58.2 mm
- net /12V_in_protected: track 94.8 -> 99.5 mm
- net +3V3: track 57.0 -> 60.9 mm
- net /throttle_in_3V3: track 63.6 -> 62.3 mm

Commit message: kicad-pcb-layout-v1.0.7
Routing:
- net /CAN_TX: track 17.4 -> 18.3 mm
- net /brake_in_3V3: track 83.9 -> 84.6 mm
- net /CAN_RX: track 20.0 -> 20.8 mm
- net /throttle_in_3V3: track 62.3 -> 61.6 mm
Changed lines of the file:
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@@
+	)
+	(segment
+		(start 119.148 89.782939)
+		(end 119.148 84.1775)
+		(width 0.25)
+		(layer "F.Cu")
+		(net 12)
 	)
 	(segment
@@
 	)
 	(segment
-		(start 119.145 84.1805)
+		(start 119.148 90.247061)
+		(end 119.145 90.244061)
+		(width 0.25)
+		(layer "F.Cu")
+		(net 12)
+	)
+	(segment
+		(start 119.148 84.1775)
 		(end 120.8355 82.49)
 		(width 0.25)
@@
 	)
 	(segment
-		(start 119.145 96.278712)
-		(end 119.145 84.1805)
+		(start 119.148 96.281712)
+		(end 119.148 90.247061)
 		(width 0.25)
 		(layer "F.Cu")
@@
 	)
 	(segment
+		(start 119.145 90.244061)
+		(end 119.145 89.785939)
+		(width 0.25)
+		(layer "F.Cu")
+		(net 12)
+	)
+	(segment
 		(start 122.698 99.831712)
-		(end 119.145 96.278712)
+		(end 119.148 96.281712)
+		(width 0.25)
+		(layer "F.Cu")
+		(net 12)
+	)
+	(segment
+		(start 119.145 89.785939)
+		(end 119.148 89.782939)
 		(width 0.25)
 		(layer "F.Cu")
@@
 	)
 	(segment
-		(start 148.2355 84.715)
-		(end 148.2355 87.339845)
-		(width 0.25)
-		(layer "F.Cu")
-		(net 20)
-	)
-	(segment
 		(start 170.901 85.687)
 		(end 175.37 85.687)
@@
 	)
 	(segment
+		(start 147.848 87.315)
+		(end 147.848 85.1025)
+		(width 0.6)
+		(layer "F.Cu")
+		(net 20)
+	)
+	(segment
+		(start 147.848 87.315)
+		(end 147.848 88.8275)
+		(width 0.6)
+		(layer "F.Cu")
+		(net 20)
+	)
+	(segment
 		(start 174.198 91.915)
 		(end 177.998 95.715)
 		(width 0.25)
+		(layer "F.Cu")
+		(net 20)
+	)
+	(segment
+		(start 147.848 88.8275)
+		(end 148.1355 89.115)
+		(width 0.6)
 		(layer "F.Cu")
 		(net 20)
@@
 	)
 	(segment
-		(start 148.2355 87.339845)
-		(end 147.9355 87.639845)
-		(width 0.25)
-		(layer "F.Cu")
-		(net 20)
-	)
-	(segment
-		(start 147.9355 87.639845)
-		(end 147.9355 89.202345)
-		(width 0.25)
+		(start 147.848 85.1025)
+		(end 148.2355 84.715)
+		(width 0.6)
 		(layer "F.Cu")
 		(net 20)
@@
 	)
 	(segment
-		(start 132.334 75.565)
-		(end 126.834 81.065)
-		(width 0.2)
-		(layer "F.Cu")
-		(net 23)
-	)
-	(segment
-		(start 126.834 81.065)
+		(start 128.398 81.065)
 		(end 117.768 81.065)
 		(width 0.2)
@@
 	)
 	(segment
-		(start 129.794 75.565)
-		(end 126.494 78.865)
-		(width 0.2)
-		(layer "F.Cu")
-		(net 25)
+		(start 132.334 77.129)
+		(end 128.398 81.065)
+		(width 0.2)
+		(layer "F.Cu")
+		(net 23)
+	)
+	(segment
+		(start 132.334 75.565)
+		(end 132.334 77.129)
+		(width 0.2)
+		(layer "F.Cu")
+		(net 23)
 	)
 	(segment
@@
 	)
 	(segment
-		(start 126.494 78.865)
+		(start 127.798 78.865)
 		(end 124.348 78.865)
+		(width 0.2)
+		(layer "F.Cu")
+		(net 25)
+	)
+	(segment
+		(start 129.794 75.565)
+		(end 129.794 76.869)
 		(width 0.2)
 		(layer "F.Cu")
@@
 		(start 113.958 79.275)
 		(end 113.958 81.065)
+		(width 0.2)
+		(layer "F.Cu")
+		(net 25)
+	)
+	(segment
+		(start 129.794 76.869)
+		(end 127.798 78.865)
 		(width 0.2)
 		(layer "F.Cu")
@@
 	)
 	(segment
-		(start 119.145 104.212)
-		(end 119.145 81.04575)
+		(start 124.098 109.165)
+		(end 118.848 103.915)
 		(width 0.25)
 		(layer "In2.Cu")
@@
 	)
 	(segment
-		(start 119.145 81.04575)
+		(start 118.848 103.915)
+		(end 118.848 80.74875)
+		(width 0.25)
+		(layer "In2.Cu")
+		(net 40)
+	)
+	(segment
+		(start 118.848 80.74875)
 		(end 112.498 74.39875)
 		(width 0.25)
@@
 	)
 	(segment
-		(start 124.098 109.165)
-		(end 119.145 104.212)
-		(width 0.25)
-		(layer "In2.Cu")
-		(net 40)
-	)
-	(segment
 		(start 124.323 80.04)
 		(end 119.298 80.04)
@@
 	)
 	(segment
+		(start 155.698 83.215)
+		(end 155.148 82.665)
+		(width 0.25)
+		(layer "In2.Cu")
+		(net 42)
+	)
+	(segment
+		(start 164.348 121.065)
+		(end 149.198 105.915)
+		(width 0.25)
+		(layer "In2.Cu")
+		(net 42)
+	)
+	(segment
+		(start 155.148 82.665)
+		(end 129.0855 82.665)
+		(width 0.25)
+		(layer "In2.Cu")
+		(net 42)
+	)
+	(segment
+		(start 155.698 84.165)
+		(end 155.698 83.215)
+		(width 0.25)
+		(layer "In2.Cu")
+		(net 42)
+	)
+	(segment
+		(start 149.198 105.915)
+		(end 149.198 90.665)
+		(width 0.25)
+		(layer "In2.Cu")
+		(net 42)
+	)
+	(segment
+		(start 129.0855 82.665)
+		(end 125.748 86.0025)
+		(width 0.25)
+		(layer "In2.Cu")
+		(net 42)
+	)
+	(segment
 		(start 164.348 121.315)
 		(end 164.348 121.065)
@@
 	)
 	(segment
-		(start 164.348 121.065)
-		(end 149.198 105.915)
-		(width 0.25)
-		(layer "In2.Cu")
-		(net 42)
-	)
-	(segment
-		(start 149.198 90.112598)
-		(end 155.424 83.886598)
-		(width 0.25)
-		(layer "In2.Cu")
-		(net 42)
-	)
-	(segment
-		(start 155.086588 83.039)
-		(end 128.7115 83.039)
-		(width 0.25)
-		(layer "In2.Cu")
-		(net 42)
-	)
-	(segment
-		(start 155.424 83.376412)
-		(end 155.086588 83.039)
-		(width 0.25)
-		(layer "In2.Cu")
-		(net 42)
-	)
-	(segment
-		(start 149.198 105.915)
-		(end 149.198 90.112598)
-		(width 0.25)
-		(layer "In2.Cu")
-		(net 42)
-	)
-	(segment
-		(start 128.7115 83.039)
-		(end 125.748 86.0025)
-		(width 0.25)
-		(layer "In2.Cu")
-		(net 42)
-	)
-	(segment
-		(start 155.424 83.886598)
-		(end 155.424 83.376412)
+		(start 149.198 90.665)
+		(end 155.698 84.165)
 		(width 0.25)
 		(layer "In2.Cu")
@@
 	)
 	(segment
-		(start 129.098 110.915)
-		(end 129.098 95.64)
+		(start 129.298 111.115)
+		(end 129.298 97.09)
 		(width 0.25)
 		(layer "In2.Cu")
@@
 	)
 	(segment
-		(start 125.598 93.39)
-		(end 126.848 93.39)
-		(width 0.127)
+		(start 153.698 113.165)
+		(end 131.348 113.165)
+		(width 0.25)
+		(layer "In2.Cu")
+		(net 43)
+	)
+	(segment
+		(start 129.298 97.09)
+		(end 125.598 93.39)
+		(width 0.25)
+		(layer "In2.Cu")
+		(net 43)
+	)
+	(segment
+		(start 131.348 113.165)
+		(end 129.298 111.115)
+		(width 0.25)
 		(layer "In2.Cu")
 		(net 43)
@@
 		(start 161.798 121.265)
 		(end 153.698 113.165)
-		(width 0.25)
-		(layer "In2.Cu")
-		(net 43)
-	)
-	(segment
-		(start 131.348 113.165)
-		(end 129.098 110.915)
-		(width 0.25)
-		(layer "In2.Cu")
-		(net 43)
-	)
-	(segment
-		(start 126.848 93.39)
-		(end 129.098 95.64)
-		(width 0.127)
-		(layer "In2.Cu")
-		(net 43)
-	)
-	(segment
-		(start 153.698 113.165)
-		(end 131.348 113.165)
 		(width 0.25)
 		(layer "In2.Cu")
@@
 	(segment
 		(start 143.5605 84.715)
-		(end 145.2605 84.715)
-		(width 0.25)
+		(end 143.5605 82.29)
+		(width 0.6)
 		(layer "F.Cu")
 		(net 59)
 	)
 	(segment
+		(start 145.2605 84.715)
+		(end 143.5605 84.715)
+		(width 0.6)
+		(layer "F.Cu")
+		(net 59)
+	)
+	(segment
 		(start 143.5605 82.29)
-		(end 143.5605 84.715)
-		(width 0.25)
+		(end 143.1355 81.865)
+		(width 0.6)
 		(layer "F.Cu")
 		(net 59)
-	)
-	(segment
-		(start 143.1355 81.865)
-		(end 143.5605 82.29)
-		(width 0.25)
-		(layer "F.Cu")
-		(net 59)
