File: kicad-project/project/ShieldArduino_Semaforo.kicad_sch (KiCad schematic)
At the start: 97 parts, among them IC1 TLIN1039DDFRQ1, IC2 TPS563200DDCR, IC3 MCP4901T-E_MS, J2 Conn_01x18, K1 RELAY, P1 Power, P2 Analog, P3 Digital, P4 Digital, P5 CONN_01X01, P6 CONN_01X01, P7 CONN_01X01, P8 CONN_01X01, Q1 PMOS, Q2 NMOS, Q3 NMOS, Q4 NMOS, Q5 NMOS, U1 MCP2542FD-E/MF, U3 LM4040DBZ-2.0

Commit message: kciad-schematic-tlin
Parts:
- added D10, D14: D_Small, symbol Device:D_Small
- added D7: ESD131-B1-W0201, Diode_SMD:Infineon_SG-WLL-2-3_0.58x0.28_P0.36mm, symbol Diode:ESD131-B1-W0201
- added R24: 1k, Resistor_SMD:R_0805_2012Metric_Pad1.20x1.40mm_HandSolder, symbol Device:R_Small
Connections:
- net 12V_in_protected: now also D10.2 (A); no longer C3.1, IC1.7 (VSUP)
- net GND: now also D7.2 (A2)
- net TLIN: now also R13.1, D7.1 (A1), R24.2; no longer R13.2
- net at D6.1 (K): now also R13.2; no longer R13.1
- new net: C3.1, D10.1 (K), D14.2 (A), IC1.7 (VSUP)
- new net: D14.1 (K), R24.1
Other:
- moved on the sheet: C3, C5, D6

Commit message: kicad-schematic-tlin2
Parts:
- D7: footprint Diode_SMD:Infineon_SG-WLL-2-3_0.58x0.28_P0.36mm -> footprint:SOD2613X100N
Changed lines of the file:
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@@
 	(wire
 		(pts
-			(xy 191.77 237.49) (xy 191.77 241.3)
+			(xy 191.77 237.49) (xy 191.77 242.57)
 		)
 		(stroke
@@
 	)
 	(label "12V_in_protected"
-		(at 191.77 241.3 0)
+		(at 191.77 242.57 0)
 		(effects
 			(font
@@
 			)
 		)
-		(property "Footprint" "Diode_SMD:Infineon_SG-WLL-2-3_0.58x0.28_P0.36mm"
+		(property "Footprint" "footprint:SOD2613X100N"
 			(at 167.64 209.55 0)
 			(effects
@@
 			)
 		)
-		(property "Datasheet" "https://www.infineon.com/dgdl/Infineon-ESD131-B1-W0201-DataSheet-v02_00-EN.pdf?fileId=5546d4625cc9456a015ce94850964889"
+		(property "Datasheet" "https://www.mouser.pl/ProductDetail/Texas-Instruments/ESD1LIN24DYFR?qs=rQFj71Wb1eUZk7C7kdpseg%3D%3D"
 			(at 167.64 209.55 0)
 			(effects

Commit message: kicad-schemat-work
Parts:
- removed D10, D14: D_Small, symbol Device:D_Small
- removed R24: 1k, Resistor_SMD:R_0805_2012Metric_Pad1.20x1.40mm_HandSolder, symbol Device:R_Small
Connections:
- net 12V_in_protected: now also C3.1, IC1.7 (VSUP)
Other:
- moved on the sheet: C5, D6, R13

Commit message: kicad-pcb-layout-v1.1.0
Connections:
- net +5V: no longer J2.13 (Pin_13)
- net A4(SDA): now also J2.9 (Pin_9); no longer J2.17 (Pin_17)
- net A5(SCL): now also J2.13 (Pin_13); no longer J2.18 (Pin_18)
- net GND: no longer J2.9 (Pin_9)
- no-connect marks 7 -> 9
Changed lines of the file:
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@@
 	)
 	(no_connect
+		(at 358.14 69.85)
+	)
+	(no_connect
 		(at 302.26 22.86)
 	)
@@
 	)
 	(no_connect
+		(at 358.14 72.39)
+	)
+	(no_connect
 		(at 309.88 22.86)
 	)
@@
 	(wire
 		(pts
-			(xy 349.25 69.85) (xy 358.14 69.85)
-		)
-		(stroke
-			(width 0)
-			(type default)
-		)
-	)
-	(wire
-		(pts
 			(xy 172.72 125.73) (xy 172.72 140.97)
 		)
@@
 	(wire
 		(pts
-			(xy 349.25 72.39) (xy 358.14 72.39)
-		)
-		(stroke
-			(width 0)
-			(type default)
-		)
-	)
-	(wire
-		(pts
 			(xy 76.2 36.83) (xy 76.2 40.64)
 		)
@@
 	)
 	(label "A5(SCL)"
-		(at 349.25 72.39 180)
+		(at 350.52 59.69 180)
 		(effects
 			(font
@@
 	)
 	(label "A4(SDA)"
-		(at 349.25 69.85 180)
+		(at 358.14 49.53 180)
 		(effects
 			(font
@@
 	)
 	(symbol
-		(lib_id "power:+5V")
-		(at 350.52 59.69 90)
-		(unit 1)
-		(exclude_from_sim no)
-		(in_bom yes)
-		(on_board yes)
-		(dnp no)
-		(property "Reference" "#PWR027"
-			(at 354.33 59.69 0)
-			(effects
-				(font
-					(size 1.27 1.27)
-				)
-				(hide yes)
-			)
-		)
-		(property "Value" "+5V"
-			(at 346.456 59.69 90)
-			(effects
-				(font
-					(size 1.27 1.27)
-				)
-				(justify left)
-			)
-		)
-		(property "Footprint" ""
-			(at 350.52 59.69 0)
-			(effects
-				(font
-					(size 1.27 1.27)
-				)
-				(hide yes)
-			)
-		)
-		(property "Datasheet" ""
-			(at 350.52 59.69 0)
-			(effects
-				(font
-					(size 1.27 1.27)
-				)
-				(hide yes)
-			)
-		)
-		(property "Description" "Power symbol creates a global label with name \"+5V\""
-			(at 350.52 59.69 0)
-			(effects
-				(font
-					(size 1.27 1.27)
-				)
-				(hide yes)
-			)
-		)
-		(pin "1"
-		)
-		(instances
-			(project "ShieldArduino_Semaforo"
-				(path "/9ffb0a36-b6c4-4251-92f7-01d561ef1727"
-					(reference "#PWR027")
-					(unit 1)
-				)
-			)
-		)
-	)
-	(symbol
 		(lib_id "Device:C_Small")
 		(at 88.9 38.1 0)
@@
 					(unit 1)
 				)
-			)
-		)
-	)
-	(symbol
-		(lib_id "power:GND")
-		(at 358.14 49.53 270)
-		(unit 1)
-		(exclude_from_sim no)
-		(in_bom yes)
-		(on_board yes)
-		(dnp no)
-		(property "Reference" "#PWR029"
-			(at 351.79 49.53 0)
-			(effects
-				(font
-					(size 1.27 1.27)
-				)
-				(hide yes)
-			)
-		)
-		(property "Value" "GND"
-			(at 354.838 49.276 90)
-			(effects
-				(font
-					(size 1.27 1.27)
-				)
-				(justify right)
-			)
-		)
-		(property "Footprint" ""
-			(at 358.14 49.53 0)
-			(effects
-				(font
-					(size 1.27 1.27)
-				)
-				(hide yes)
-			)
-		)
-		(property "Datasheet" ""
-			(at 358.14 49.53 0)
-			(effects
-				(font
-					(size 1.27 1.27)
-				)
-				(hide yes)
-			)
-		)
-		(property "Description" "Power symbol creates a global label with name \"GND\" , ground"
-			(at 358.14 49.53 0)
-			(effects
-				(font
-					(size 1.27 1.27)
-				)
-				(hide yes)
-			)
-		)
-		(pin "1"
-		)
-		(instances
-			(project "ShieldArduino_Semaforo"
-				(path "/9ffb0a36-b6c4-4251-92f7-01d561ef1727"
-					(reference "#PWR029")
-					(unit 1)
-				)

Commit message: kicad-pcb-layout-v1.1.1
Parts:
- added D10, D14: 6V, Diode_SMD:D_SOD-123F, symbol Device:D_TVS
- added R24, R25, R26, R27, R28, R29, R30, R31: 10k, Resistor_SMD:R_0805_2012Metric_Pad1.20x1.40mm_HandSolder, symbol Device:R_Small
Connections:
- net +3V3 is gone; now on net +3.3V: P1.4 (Pin_4), R12.1, R23.1, TP17.1
- net +3.3V: now also R24.1, R25.1, R26.1, R27.1, R28.1, R29.1, R30.1, R31.1
- net 11(**/MOSI): now also R31.2
- net 13(SCK): now also R30.2
- net A4(SDA): now also D10.1 (A1), R29.2
- net A5(SCL): now also D14.1 (A1), R28.2
- net CAN_RX: now also R26.2
- net CAN_TX: now also R27.2
- net GND: now also D10.2 (A2), D14.2 (A2)
- net UART_RX: now also R24.2
- net UART_TX: now also R25.2
Other:
- note added: "PULL UP"
- moved on the sheet: D1, D11, D12, D13, D2, D3, D4
